File: Template module/template-module.kicad_sch (KiCad schematic)
At the start: 4 parts

Commit message: Update template
Parts:
- G1: symbol 0_aurora_common:Graphic -> 0_project:Graphic
- H1, H2: symbol 0_splitkb_prime:Standoff_97730606332R -> 0_project:Standoff_97730606332R; Manufacturer Part number 97730606332R -> (none); SMD 1 -> (none)
- J1: symbol 0_splitkb_prime:vik-keyboard-connector -> 0_project:vik-keyboard-connector
Changed lines of the file:
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@@
     )
   )
-  (symbol (lib_id "0_splitkb_prime:Standoff_97730606332R") (at 157.48 130.81 270) (unit 1)
+  (symbol (lib_id "0_project:Standoff_97730606332R") (at 157.48 130.81 270) (unit 1)
     (in_bom yes) (on_board yes) (dnp no) (fields_autoplaced)
     (property "Reference" "H1" (at 161.29 129.54 90)
@@
       (effects (font (size 1.27 1.27)) hide)
     )
-    (property "Manufacturer Part number" "97730606332R" (at 157.48 130.81 0)
-      (effects (font (size 1.27 1.27)) hide)
-    )
-    (property "Description" "Standoff M1.6 H6mm 2mm depth" (at 157.48 130.81 0)
-      (effects (font (size 1.27 1.27)) hide)
-    )
-    (property "SMD" "1" (at 157.48 130.81 0)
-      (effects (font (size 1.27 1.27)) hide)
-    )
-    (property "THT" "" (at 157.48 130.81 0)
-      (effects (font (size 1.27 1.27)) hide)
-    )
-    (property "Original" "" (at 157.48 130.81 0)
-      (effects (font (size 1.27 1.27)) hide)
-    )
-    (property "Elecrow PN" "" (at 157.48 130.81 0)
-      (effects (font (size 1.27 1.27)) hide)
-    )
-    (property "Note" "" (at 157.48 130.81 0)
-      (effects (font (size 1.27 1.27)) hide)
-    )
     (pin "1")
     (instances
@@
     )
   )
-  (symbol (lib_id "0_splitkb_prime:vik-keyboard-connector") (at 154.94 96.52 0) (unit 1)
+  (symbol (lib_id "0_project:vik-keyboard-connector") (at 154.94 96.52 0) (unit 1)
     (in_bom yes) (on_board yes) (dnp no)
     (property "Reference" "J1" (at 172.72 96.52 0)
@@
       (effects (font (size 1.27 1.27)))
     )
-    (property "Footprint" "0_project:vik-module-connector" (at 154.94 90.17 0)
+    (property "Footprint" "0_project:vik-module-connector" (at 154.94 78.994 0)
       (effects (font (size 1.27 1.27)) hide)
     )
@@
     )
   )
-  (symbol (lib_id "0_splitkb_prime:Standoff_97730606332R") (at 157.48 135.89 270) (unit 1)
+  (symbol (lib_id "0_project:Standoff_97730606332R") (at 157.48 135.89 270) (unit 1)
     (in_bom yes) (on_board yes) (dnp no) (fields_autoplaced)
     (property "Reference" "H2" (at 161.29 134.62 90)
@@
       (effects (font (size 1.27 1.27)) hide)
     )
-    (property "Manufacturer Part number" "97730606332R" (at 157.48 135.89 0)
-      (effects (font (size 1.27 1.27)) hide)
-    )
-    (property "Description" "Standoff M1.6 H6mm 2mm depth" (at 157.48 135.89 0)
-      (effects (font (size 1.27 1.27)) hide)
-    )
-    (property "SMD" "1" (at 157.48 135.89 0)
-      (effects (font (size 1.27 1.27)) hide)
-    )
-    (property "THT" "" (at 157.48 135.89 0)
-      (effects (font (size 1.27 1.27)) hide)
-    )
-    (property "Original" "" (at 157.48 135.89 0)
-      (effects (font (size 1.27 1.27)) hide)
-    )
-    (property "Elecrow PN" "" (at 157.48 135.89 0)
-      (effects (font (size 1.27 1.27)) hide)
-    )
-    (property "Note" "" (at 157.48 135.89 0)
-      (effects (font (size 1.27 1.27)) hide)
-    )
     (pin "1")
     (instances
@@
     )
   )
-  (symbol (lib_id "0_aurora_common:Graphic") (at 157.48 142.24 0) (unit 1)
+  (symbol (lib_id "0_project:Graphic") (at 157.48 142.24 0) (unit 1)
     (in_bom no) (on_board yes) (dnp no) (fields_autoplaced)
     (property "Reference" "G1" (at 161.29 140.9717 0)
